File: usbB_isp.sch (EAGLE design)
At the start: 12 parts, among them IC1 788TV, IC2 TINY13-20PU, X1 PN61729-S

Commit message: reroute, using 16 mil wires
Connections:
- net N$10 renamed MOSI
Changed lines of the file:
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@@
 </segment>
 </net>
-<net name="N$10" class="0">
+<net name="MOSI" class="0">
 <segment>
 <pinref part="IC2" gate="G$1" pin="PB0/PCINT0/AIN0/OC0A/MOSI"/>
